File: connectors.kicad_sch (KiCad schematic)
At the start: 7 parts, among them J1 MicroFit_1x4, J2 MicroFit_1x4

Commit message: schematic and routing updated
Parts:
- renumbered C6 to C8, C7 to C9
Changed lines of the file:
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@@
 	(title_block
 		(title "LEOS Connectors")
-		(date "2026-08-04")
-		(rev "3.0")
+		(date "2026-10-05")
+		(rev "1.0")
 		(company "VIP Lightning From the Edge of Space")
 	)
@@
 		(in_pos_files yes)
 		(dnp no)
-		(property "Reference" "C6"
+		(property "Reference" "C8"
 			(at 114.808 50.038 0)
 			(show_name no)
@@
 		)
 		(instances
-			(project "LEOS-stack-template"
+			(project "LEOS-F26-radio"
 				(path "/3703ddf2-8141-438d-86a8-1eaec9672d0d/341d819d-3d1a-4f8b-94f1-4c6aaa16d806"
-					(reference "C6")
+					(reference "C8")
 					(unit 1)
 				)
@@
 		)
 		(instances
-			(project "LEOS-stack-template"
+			(project "LEOS-F26-radio"
 				(path "/3703ddf2-8141-438d-86a8-1eaec9672d0d/341d819d-3d1a-4f8b-94f1-4c6aaa16d806"
 					(reference "J1")
@@
 		)
 		(instances
-			(project "LEOS-stack-template"
+			(project "LEOS-F26-radio"
 				(path "/3703ddf2-8141-438d-86a8-1eaec9672d0d/341d819d-3d1a-4f8b-94f1-4c6aaa16d806"
 					(reference "#PWR018")
@@
 		)
 		(instances
-			(project "LEOS-stack-template"
+			(project "LEOS-F26-radio"
 				(path "/3703ddf2-8141-438d-86a8-1eaec9672d0d/341d819d-3d1a-4f8b-94f1-4c6aaa16d806"
 					(reference "#PWR017")
@@
 		)
 		(instances
-			(project "LEOS-stack-template"
+			(project "LEOS-F26-radio"
 				(path "/3703ddf2-8141-438d-86a8-1eaec9672d0d/341d819d-3d1a-4f8b-94f1-4c6aaa16d806"
 					(reference "#FLG01")
@@
 		(in_pos_files yes)
 		(dnp no)
-		(property "Reference" "C7"
+		(property "Reference" "C9"
 			(at 122.428 50.038 0)
 			(show_name no)
@@
 		)
 		(instances
-			(project "LEOS-stack-template"
+			(project "LEOS-F26-radio"
 				(path "/3703ddf2-8141-438d-86a8-1eaec9672d0d/341d819d-3d1a-4f8b-94f1-4c6aaa16d806"
-					(reference "C7")
+					(reference "C9")
 					(unit 1)
 				)
@@
 		)
 		(instances
-			(project "LEOS-stack-template"
+			(project "LEOS-F26-radio"
 				(path "/3703ddf2-8141-438d-86a8-1eaec9672d0d/341d819d-3d1a-4f8b-94f1-4c6aaa16d806"
 					(reference "R1")
@@
 		)
 		(instances
-			(project "LEOS-stack-template"
+			(project "LEOS-F26-radio"
 				(path "/3703ddf2-8141-438d-86a8-1eaec9672d0d/341d819d-3d1a-4f8b-94f1-4c6aaa16d806"
 					(reference "J2")
@@
 		)
 		(instances
-			(project "LEOS-stack-template"
+			(project "LEOS-F26-radio"
 				(path "/3703ddf2-8141-438d-86a8-1eaec9672d0d/341d819d-3d1a-4f8b-94f1-4c6aaa16d806"
 					(reference "TP4")
@@
 		)
 		(instances
-			(project "LEOS-stack-template"
+			(project "LEOS-F26-radio"
 				(path "/3703ddf2-8141-438d-86a8-1eaec9672d0d/341d819d-3d1a-4f8b-94f1-4c6aaa16d806"
 					(reference "#PWR019")
@@
 		)
 		(instances
-			(project "LEOS-stack-template"
+			(project "LEOS-F26-radio"
 				(path "/3703ddf2-8141-438d-86a8-1eaec9672d0d/341d819d-3d1a-4f8b-94f1-4c6aaa16d806"
 					(reference "TP3")
@@
 		)
 		(instances
-			(project "LEOS-stack-template"
+			(project "LEOS-F26-radio"
 				(path "/3703ddf2-8141-438d-86a8-1eaec9672d0d/341d819d-3d1a-4f8b-94f1-4c6aaa16d806"
 					(reference "#PWR020")
